Commit message: Aliengo visualization complete

File: robots/xpp_aliengo/urdf/aliengo.urdf (robot description, URDF)
Before this commit: robot hyq, 0 links, 0 joints
Links:
- added link FL_calf, mass 0.207; collision box size=0.25 0.0208 0.016; visual mesh filename=package://xpp_aliengo/meshes/calf.stl scale=1 1 1
- added link FL_foot, mass 0.06; collision sphere radius=0.0265; visual sphere radius=0.0165
- added link FL_hip, mass 1.993; collision cylinder length=0.0418 radius=0.046; visual mesh filename=package://xpp_aliengo/meshes/hip.stl scale=1 1 1
- added link FL_thigh, mass 0.639; collision box size=0.25 0.0374 0.043; visual mesh filename=package://xpp_aliengo/meshes/thigh.stl scale=1 1 1
- added link FR_calf, mass 0.207; collision box size=0.25 0.0208 0.016; visual mesh filename=package://xpp_aliengo/meshes/calf.stl scale=1 1 1
- added link FR_foot, mass 0.06; collision sphere radius=0.0265; visual sphere radius=0.0165
- added link FR_hip, mass 1.993; collision cylinder length=0.0418 radius=0.046; visual mesh filename=package://xpp_aliengo/meshes/hip.stl scale=1 1 1
- added link FR_thigh, mass 0.639; collision box size=0.25 0.0374 0.043; visual mesh filename=package://xpp_aliengo/meshes/thigh_mirror.stl scale=1 1 1
- added link RL_calf, mass 0.207; collision box size=0.25 0.0208 0.016; visual mesh filename=package://xpp_aliengo/meshes/calf.stl scale=1 1 1
- added link RL_foot, mass 0.06; collision sphere radius=0.0265; visual sphere radius=0.0165
- added link RL_hip, mass 1.993; collision cylinder length=0.0418 radius=0.046; visual mesh filename=package://xpp_aliengo/meshes/hip.stl scale=1 1 1
- added link RL_thigh, mass 0.639; collision box size=0.25 0.0374 0.043; visual mesh filename=package://xpp_aliengo/meshes/thigh.stl scale=1 1 1
- added link RR_calf, mass 0.207; collision box size=0.25 0.0208 0.016; visual mesh filename=package://xpp_aliengo/meshes/calf.stl scale=1 1 1
- added link RR_foot, mass 0.06; collision sphere radius=0.0265; visual sphere radius=0.0165
- added link RR_hip, mass 1.993; collision cylinder length=0.0418 radius=0.046; visual mesh filename=package://xpp_aliengo/meshes/hip.stl scale=1 1 1
- added link RR_thigh, mass 0.639; collision box size=0.25 0.0374 0.043; visual mesh filename=package://xpp_aliengo/meshes/thigh_mirror.stl scale=1 1 1
- added link base; visual box size=0.001 0.001 0.001
- added link imu_link, mass 0.001; collision box size=.001 .001 .001; visual box size=0.001 0.001 0.001
- added link trunk, mass 9.041; collision box size=0.647 0.15 0.112; visual mesh filename=package://xpp_aliengo/meshes/trunk.stl scale=1 1 1
Joints:
- added joint FL_calf_joint: type revolute, parent FL_thigh, child FL_calf, origin xyz=0 0 -0.25 rpy=0 0 0, axis 0 1 0, limit lower=-2.77507351067 upper=-0.645771823238 effort=44.4 velocity=40
- added joint FL_foot_fixed: type fixed, parent FL_calf, child FL_foot, origin xyz=0 0 -0.25 rpy=0 0 0
- added joint FL_hip_joint: type revolute, parent trunk, child FL_hip, origin xyz=0.2399 0.051 0 rpy=0 0 0, axis 1 0 0, limit lower=-1.2217304764 upper=1.2217304764 effort=44.4 velocity=40
- added joint FL_thigh_joint: type continuous, parent FL_hip, child FL_thigh, origin xyz=0 0.083 0 rpy=0 0 0, axis 0 1 0, limit effort=44.4 velocity=40
- added joint FR_calf_joint: type revolute, parent FR_thigh, child FR_calf, origin xyz=0 0 -0.25 rpy=0 0 0, axis 0 1 0, limit lower=-2.77507351067 upper=-0.645771823238 effort=44.4 velocity=40
- added joint FR_foot_fixed: type fixed, parent FR_calf, child FR_foot, origin xyz=0 0 -0.25 rpy=0 0 0
- added joint FR_hip_joint: type revolute, parent trunk, child FR_hip, origin xyz=0.2399 -0.051 0 rpy=0 0 0, axis 1 0 0, limit lower=-1.2217304764 upper=1.2217304764 effort=44.4 velocity=40
- added joint FR_thigh_joint: type continuous, parent FR_hip, child FR_thigh, origin xyz=0 -0.083 0 rpy=0 0 0, axis 0 1 0, limit effort=44.4 velocity=40
- added joint RL_calf_joint: type revolute, parent RL_thigh, child RL_calf, origin xyz=0 0 -0.25 rpy=0 0 0, axis 0 1 0, limit lower=-2.77507351067 upper=-0.645771823238 effort=44.4 velocity=40
- added joint RL_foot_fixed: type fixed, parent RL_calf, child RL_foot, origin xyz=0 0 -0.25 rpy=0 0 0
- added joint RL_hip_joint: type revolute, parent trunk, child RL_hip, origin xyz=-0.2399 0.051 0 rpy=0 0 0, axis 1 0 0, limit lower=-1.2217304764 upper=1.2217304764 effort=44.4 velocity=40
- added joint RL_thigh_joint: type continuous, parent RL_hip, child RL_thigh, origin xyz=0 0.083 0 rpy=0 0 0, axis 0 1 0, limit effort=44.4 velocity=40
- added joint RR_calf_joint: type revolute, parent RR_thigh, child RR_calf, origin xyz=0 0 -0.25 rpy=0 0 0, axis 0 1 0, limit lower=-2.77507351067 upper=-0.645771823238 effort=44.4 velocity=40
- added joint RR_foot_fixed: type fixed, parent RR_calf, child RR_foot, origin xyz=0 0 -0.25 rpy=0 0 0
- added joint RR_hip_joint: type revolute, parent trunk, child RR_hip, origin xyz=-0.2399 -0.051 0 rpy=0 0 0, axis 1 0 0, limit lower=-1.2217304764 upper=1.2217304764 effort=44.4 velocity=40
- added joint RR_thigh_joint: type continuous, parent RR_hip, child RR_thigh, origin xyz=0 -0.083 0 rpy=0 0 0, axis 0 1 0, limit effort=44.4 velocity=40
- added joint floating_base: type fixed, parent base, child trunk, origin xyz=0 0 0 rpy=0 0 0
- added joint imu_joint: type fixed, parent trunk, child imu_link, origin xyz=0 0 0 rpy=0 0 0
